File: Oscillator.sch (KiCad schematic (older format))
At the start: 12 parts, among them U5 LT1016, Y1 13.56 Mhz

Commit message: updated csv
Parts:
- C12: Mouser 581-08051A870FAT2A -> 81-GCM21A5C2J910JX1D
Changed lines of the file:
@@
 F 2 "Capacitor_SMD:C_0805_2012Metric_Pad1.15x1.40mm_HandSolder" H 7988 3700 50  0001 C CNN
 F 3 "~" H 7950 3850 50  0001 C CNN
-F 4 "581-08051A870FAT2A" H 7950 3850 50  0001 C CNN "Mouser"
+F 4 "81-GCM21A5C2J910JX1D" H 7950 3850 50  0001 C CNN "Mouser"
 	1    7950 3850
 	1    0    0    -1
